File: backplane2/OSH_Park_2_layer.kicad_pcb (KiCad board)
At the start: 2 copper layers, 2 parts

Commit message: working on board design
Parts:
- removed N1: OHWLOGO, Symbols:OSHW-Symbol_6.7x6mm_SilkScreen
- added C1: CP, Capacitor_THT:CP_Radial_D8.0mm_P2.50mm, F.Cu at (205.7, 75.2)
- added D1: LED, LED_THT:LED_D5.0mm, F.Cu at (205.6, 96.0)
- added J1: Conn_02x40_Odd_Even, Connector_PinHeader_2.54mm:PinHeader_2x40_P2.54mm_Vertical, F.Cu at (50.8, 50.8)
- added J10: Conn_01x40, Connector_PinHeader_2.54mm:PinHeader_1x40_P2.54mm_Vertical, F.Cu at (177.8, 50.8)
- added J11: Conn_01x40, Connector_PinHeader_2.54mm:PinHeader_1x40_P2.54mm_Vertical, F.Cu at (180.3, 50.8)
- added J12: Conn_01x40, Connector_PinHeader_2.54mm:PinHeader_1x40_P2.54mm_Vertical, F.Cu at (182.9, 50.8)
- added J13: Conn_01x40, Connector_PinHeader_2.54mm:PinHeader_1x40_P2.54mm_Vertical, F.Cu at (185.4, 50.8)
- added J14: Conn_01x40, Connector_PinHeader_2.54mm:PinHeader_1x40_P2.54mm_Vertical, F.Cu at (188.0, 50.8)
- added J15: Conn_01x40, Connector_PinHeader_2.54mm:PinHeader_1x40_P2.54mm_Vertical, F.Cu at (190.5, 50.8)
- added J16: Conn_01x40, Connector_PinHeader_2.54mm:PinHeader_1x40_P2.54mm_Vertical, F.Cu at (193.0, 50.8)
- added J17: Conn_01x40, Connector_PinHeader_2.54mm:PinHeader_1x40_P2.54mm_Vertical, F.Cu at (195.6, 50.8)
- added J18: Conn_01x40, Connector_PinHeader_2.54mm:PinHeader_1x40_P2.54mm_Vertical, F.Cu at (198.1, 50.8)
- added J19: Conn_01x40, Connector_PinHeader_2.54mm:PinHeader_1x40_P2.54mm_Vertical, F.Cu at (200.7, 50.8)
- added J2: Conn_02x40_Odd_Even, Connector_PinHeader_2.54mm:PinHeader_2x40_P2.54mm_Vertical, F.Cu at (69.8, 50.8)
- added J20: Conn_01x02, Connector_PinHeader_2.54mm:PinHeader_1x02_P2.54mm_Vertical, F.Cu at (206.8, 82.5)
- added J21: OSTTA020161, OSTTA020161:OST_OSTTA020161, F.Cu at (206.9, 64.3)
- added J3: Conn_02x40_Odd_Even, Connector_PinHeader_2.54mm:PinHeader_2x40_P2.54mm_Vertical, F.Cu at (88.9, 50.8)
- added J4: Conn_02x40_Odd_Even, Connector_PinHeader_2.54mm:PinHeader_2x40_P2.54mm_Vertical, F.Cu at (108.0, 50.8)
- added J5: Conn_02x40_Odd_Even, Connector_PinHeader_2.54mm:PinHeader_2x40_P2.54mm_Vertical, F.Cu at (127.0, 50.8)
- added J6: Conn_02x40_Odd_Even, Connector_PinHeader_2.54mm:PinHeader_2x40_P2.54mm_Vertical, F.Cu at (146.1, 50.8)
- added J7: Conn_02x40_Odd_Even, Connector_PinHeader_2.54mm:PinHeader_2x40_P2.54mm_Vertical, F.Cu at (165.1, 50.8)
- added R1: R, Resistor_THT:R_Axial_DIN0204_L3.6mm_D1.6mm_P7.62mm_Horizontal, F.Cu at (203.2, 90.7)
- added REF**: MountingHole_3.2mm_M3_Pad, MountingHole:MountingHole_3.2mm_M3_Pad, F.Cu at (207.0, 147.3)
- added REF**: MountingHole_3.2mm_M3_Pad, MountingHole:MountingHole_3.2mm_M3_Pad, F.Cu at (207.0, 53.3)
- added REF**: MountingHole_3.2mm_M3_Pad, MountingHole:MountingHole_3.2mm_M3_Pad, F.Cu at (44.5, 147.3)
- added REF**: MountingHole_3.2mm_M3_Pad, MountingHole:MountingHole_3.2mm_M3_Pad, F.Cu at (44.5, 53.3)
Other:
- board text added: "+"
- board text added: "-"
