File: backplane2/OSH_Park_2_layer.sch (KiCad schematic (older format))
At the start: 22 parts, among them J1 Conn_02x40_Odd_Even, J10 Conn_01x40, J11 Conn_01x40, J12 Conn_01x40, J13 Conn_01x40, J14 Conn_01x40, J15 Conn_01x40, J16 Conn_01x40, J17 Conn_01x40, J18 Conn_01x40, J19 Conn_01x40, J2 Conn_02x40_Odd_Even, J20 Conn_01x02, J21 OSTTA020161, J3 Conn_02x40_Odd_Even, J4 Conn_02x40_Odd_Even, J5 Conn_02x40_Odd_Even, J6 Conn_02x40_Odd_Even, J7 Conn_02x40_Odd_Even

Commit message: working on board design
Parts:
- C1: footprint Capacitor_THT:CP_Radial_D10.0mm_P5.00mm -> Capacitor_THT:CP_Radial_D8.0mm_P2.50mm
- J1, J2, J3, J4, J5, J6, J7: footprint Connector_PinSocket_2.54mm:PinSocket_2x40_P2.54mm_Vertical -> Connector_PinHeader_2.54mm:PinHeader_2x40_P2.54mm_Vertical
- J10, J11, J12, J13, J14, J15, J16, J17, J18, J19: footprint Connector_PinSocket_2.54mm:PinSocket_1x40_P2.54mm_Vertical -> Connector_PinHeader_2.54mm:PinHeader_1x40_P2.54mm_Vertical
- J20: footprint Connector_PinSocket_2.54mm:PinSocket_1x40_P2.54mm_Vertical -> Connector_PinHeader_2.54mm:PinHeader_1x02_P2.54mm_Vertical
Changed lines of the file:
@@
 F 0 "J1" H 1700 4967 50  0000 C CNN
 F 1 "Conn_02x40_Odd_Even" H 1700 4876 50  0000 C CNN
-F 2 "Connector_PinSocket_2.54mm:PinSocket_2x40_P2.54mm_Vertical" H 1650 2850 50  0001 C CNN
+F 2 "Connector_PinHeader_2.54mm:PinHeader_2x40_P2.54mm_Vertical" H 1650 2850 50  0001 C CNN
 F 3 "~" H 1650 2850 50  0001 C CNN
 	1    1650 2850
@@
 F 0 "J2" H 2950 4967 50  0000 C CNN
 F 1 "Conn_02x40_Odd_Even" H 2950 4876 50  0000 C CNN
-F 2 "Connector_PinSocket_2.54mm:PinSocket_2x40_P2.54mm_Vertical" H 2900 2850 50  0001 C CNN
+F 2 "Connector_PinHeader_2.54mm:PinHeader_2x40_P2.54mm_Vertical" H 2900 2850 50  0001 C CNN
 F 3 "~" H 2900 2850 50  0001 C CNN
 	1    2900 2850
@@
 F 0 "J3" H 4200 4967 50  0000 C CNN
 F 1 "Conn_02x40_Odd_Even" H 4200 4876 50  0000 C CNN
-F 2 "Connector_PinSocket_2.54mm:PinSocket_2x40_P2.54mm_Vertical" H 4150 2850 50  0001 C CNN
+F 2 "Connector_PinHeader_2.54mm:PinHeader_2x40_P2.54mm_Vertical" H 4150 2850 50  0001 C CNN
 F 3 "~" H 4150 2850 50  0001 C CNN
 	1    4150 2850
@@
 F 0 "J4" H 5450 4967 50  0000 C CNN
 F 1 "Conn_02x40_Odd_Even" H 5450 4876 50  0000 C CNN
-F 2 "Connector_PinSocket_2.54mm:PinSocket_2x40_P2.54mm_Vertical" H 5400 2850 50  0001 C CNN
+F 2 "Connector_PinHeader_2.54mm:PinHeader_2x40_P2.54mm_Vertical" H 5400 2850 50  0001 C CNN
 F 3 "~" H 5400 2850 50  0001 C CNN
 	1    5400 2850
@@
 F 0 "J5" H 6700 4967 50  0000 C CNN
 F 1 "Conn_02x40_Odd_Even" H 6700 4876 50  0000 C CNN
-F 2 "Connector_PinSocket_2.54mm:PinSocket_2x40_P2.54mm_Vertical" H 6650 2850 50  0001 C CNN
+F 2 "Connector_PinHeader_2.54mm:PinHeader_2x40_P2.54mm_Vertical" H 6650 2850 50  0001 C CNN
 F 3 "~" H 6650 2850 50  0001 C CNN
 	1    6650 2850
@@
 F 0 "J6" H 7950 4967 50  0000 C CNN
 F 1 "Conn_02x40_Odd_Even" H 7950 4876 50  0000 C CNN
-F 2 "Connector_PinSocket_2.54mm:PinSocket_2x40_P2.54mm_Vertical" H 7900 2850 50  0001 C CNN
+F 2 "Connector_PinHeader_2.54mm:PinHeader_2x40_P2.54mm_Vertical" H 7900 2850 50  0001 C CNN
 F 3 "~" H 7900 2850 50  0001 C CNN
 	1    7900 2850
@@
 F 0 "J7" H 9200 4967 50  0000 C CNN
 F 1 "Conn_02x40_Odd_Even" H 9200 4876 50  0000 C CNN
-F 2 "Connector_PinSocket_2.54mm:PinSocket_2x40_P2.54mm_Vertical" H 9150 2850 50  0001 C CNN
+F 2 "Connector_PinHeader_2.54mm:PinHeader_2x40_P2.54mm_Vertical" H 9150 2850 50  0001 C CNN
 F 3 "~" H 9150 2850 50  0001 C CNN
 	1    9150 2850
@@
 F 0 "J10" V 2850 7400 50  0000 C CNN
 F 1 "Conn_01x40" V 2950 7550 50  0000 C CNN
-F 2 "Connector_PinSocket_2.54mm:PinSocket_1x40_P2.54mm_Vertical" H 3050 5350 50  0001 C CNN
+F 2 "Connector_PinHeader_2.54mm:PinHeader_1x40_P2.54mm_Vertical" H 3050 5350 50  0001 C CNN
 F 3 "~" H 3050 5350 50  0001 C CNN
 	1    3050 5350
@@
 F 0 "J11" V 2850 7700 50  0000 C CNN
 F 1 "Conn_01x40" V 2950 7850 50  0000 C CNN
-F 2 "Connector_PinSocket_2.54mm:PinSocket_1x40_P2.54mm_Vertical" H 3050 5650 50  0001 C CNN
+F 2 "Connector_PinHeader_2.54mm:PinHeader_1x40_P2.54mm_Vertical" H 3050 5650 50  0001 C CNN
 F 3 "~" H 3050 5650 50  0001 C CNN
 	1    3050 5650
@@
 F 0 "J12" V 2850 8000 50  0000 C CNN
 F 1 "Conn_01x40" V 2950 8150 50  0000 C CNN
-F 2 "Connector_PinSocket_2.54mm:PinSocket_1x40_P2.54mm_Vertical" H 3050 5950 50  0001 C CNN
+F 2 "Connector_PinHeader_2.54mm:PinHeader_1x40_P2.54mm_Vertical" H 3050 5950 50  0001 C CNN
 F 3 "~" H 3050 5950 50  0001 C CNN
 	1    3050 5950
@@
 F 0 "J13" V 2850 8300 50  0000 C CNN
 F 1 "Conn_01x40" V 2950 8450 50  0000 C CNN
-F 2 "Connector_PinSocket_2.54mm:PinSocket_1x40_P2.54mm_Vertical" H 3050 6250 50  0001 C CNN
+F 2 "Connector_PinHeader_2.54mm:PinHeader_1x40_P2.54mm_Vertical" H 3050 6250 50  0001 C CNN
 F 3 "~" H 3050 6250 50  0001 C CNN
 	1    3050 6250
@@
 F 0 "J14" V 2850 8600 50  0000 C CNN
 F 1 "Conn_01x40" V 2950 8750 50  0000 C CNN
-F 2 "Connector_PinSocket_2.54mm:PinSocket_1x40_P2.54mm_Vertical" H 3050 6550 50  0001 C CNN
+F 2 "Connector_PinHeader_2.54mm:PinHeader_1x40_P2.54mm_Vertical" H 3050 6550 50  0001 C CNN
 F 3 "~" H 3050 6550 50  0001 C CNN
 	1    3050 6550
@@
 F 0 "J15" V 2850 8900 50  0000 C CNN
 F 1 "Conn_01x40" V 2950 9050 50  0000 C CNN
-F 2 "Connector_PinSocket_2.54mm:PinSocket_1x40_P2.54mm_Vertical" H 3050 6850 50  0001 C CNN
+F 2 "Connector_PinHeader_2.54mm:PinHeader_1x40_P2.54mm_Vertical" H 3050 6850 50  0001 C CNN
 F 3 "~" H 3050 6850 50  0001 C CNN
 	1    3050 6850
@@
 F 0 "J16" V 2850 9200 50  0000 C CNN
 F 1 "Conn_01x40" V 2950 9350 50  0000 C CNN
-F 2 "Connector_PinSocket_2.54mm:PinSocket_1x40_P2.54mm_Vertical" H 3050 7150 50  0001 C CNN
+F 2 "Connector_PinHeader_2.54mm:PinHeader_1x40_P2.54mm_Vertical" H 3050 7150 50  0001 C CNN
 F 3 "~" H 3050 7150 50  0001 C CNN
 	1    3050 7150
@@
 F 0 "J17" V 2850 9500 50  0000 C CNN
 F 1 "Conn_01x40" V 2950 9650 50  0000 C CNN
-F 2 "Connector_PinSocket_2.54mm:PinSocket_1x40_P2.54mm_Vertical" H 3050 7450 50  0001 C CNN
+F 2 "Connector_PinHeader_2.54mm:PinHeader_1x40_P2.54mm_Vertical" H 3050 7450 50  0001 C CNN
 F 3 "~" H 3050 7450 50  0001 C CNN
 	1    3050 7450
@@
 F 0 "J18" V 7600 7400 50  0000 C CNN
 F 1 "Conn_01x40" V 7700 7550 50  0000 C CNN
-F 2 "Connector_PinSocket_2.54mm:PinSocket_1x40_P2.54mm_Vertical" H 7800 5350 50  0001 C CNN
+F 2 "Connector_PinHeader_2.54mm:PinHeader_1x40_P2.54mm_Vertical" H 7800 5350 50  0001 C CNN
 F 3 "~" H 7800 5350 50  0001 C CNN
 	1    7800 5350
@@
 F 0 "J19" V 7600 7700 50  0000 C CNN
 F 1 "Conn_01x40" V 7700 7850 50  0000 C CNN
-F 2 "Connector_PinSocket_2.54mm:PinSocket_1x40_P2.54mm_Vertical" H 7800 5650 50  0001 C CNN
+F 2 "Connector_PinHeader_2.54mm:PinHeader_1x40_P2.54mm_Vertical" H 7800 5650 50  0001 C CNN
 F 3 "~" H 7800 5650 50  0001 C CNN
 	1    7800 5650
@@
 F 0 "J20" H 7950 6350 50  0000 C CNN
 F 1 "Conn_01x02" H 7950 6250 50  0000 C CNN
-F 2 "Connector_PinSocket_2.54mm:PinSocket_1x40_P2.54mm_Vertical" H 7950 6100 50  0001 C CNN
+F 2 "Connector_PinHeader_2.54mm:PinHeader_1x02_P2.54mm_Vertical" H 7950 6100 50  0001 C CNN
 F 3 "~" H 7950 6100 50  0001 C CNN
 	1    7950 6100
@@
 F 0 "C1" H 8968 6296 50  0000 L CNN
 F 1 "CP" H 8968 6205 50  0000 L CNN
-F 2 "Capacitor_THT:CP_Radial_D10.0mm_P5.00mm" H 8888 6100 50  0001 C CNN
+F 2 "Capacitor_THT:CP_Radial_D8.0mm_P2.50mm" H 8888 6100 50  0001 C CNN
 F 3 "" H 8850 6250 50  0001 C CNN
 	1    8850 6250
